Commit message: add linkhou chassis

File: xacro/body_sinopec.xacro (robot description, xacro)
@@ -1,4 +1,4 @@
 <?xml version="1.0"?>
-<robot name="FiveAges W2 Body" xmlns:xacro="http://www.ros.org/wiki/xacro">
+<robot name="FiveAges W2" xmlns:xacro="http://www.ros.org/wiki/xacro">
 	<xacro:property name="PI" value="3.1415926535897931"/>
 	<link name="body_base">
@@ -16,5 +16,5 @@
 		<visual>
 			<geometry>
-				<mesh filename="file://$(find fiveages_body_description)/meshes/base.glb"/>
+				<mesh filename="file://$(find fiveages_w2_description)/meshes/body/base.glb"/>
 			</geometry>
 		</visual>
@@ -39,5 +39,5 @@
 		<visual>
 			<geometry>
-				<mesh filename="file://$(find fiveages_body_description)/meshes/link1.glb"/>
+				<mesh filename="file://$(find fiveages_w2_description)/meshes/body/link1.glb"/>
 			</geometry>
 		</visual>
@@ -53,5 +53,5 @@
 		<child link="body_link1"/>
 		<axis xyz="0 1 0"/>
-		<limit lower="-1.352633" upper="0.567" effort="500" velocity="1"/>
+		<limit lower="-${PI*70/180}" upper="${PI*30/180}" effort="100" velocity="1"/>
 	</joint>
 	<link name="body_link2">
@@ -69,5 +69,5 @@
 		<visual>
 			<geometry>
-				<mesh filename="file://$(find fiveages_body_description)/meshes/link2.glb"/>
+				<mesh filename="file://$(find fiveages_w2_description)/meshes/body/link2.glb"/>
 			</geometry>
 		</visual>
@@ -84,5 +84,5 @@
 		<child link="body_link2"/>
 		<axis xyz="0 -1 0"/>
-		<limit lower="-2.66" upper="1.605" effort="500" velocity="1"/>
+		<limit lower="-${PI*120/180}" upper="${PI*90/180}" effort="100" velocity="1"/>
 	</joint>
 	<link name="body_link3">
@@ -100,5 +100,5 @@
 		<visual>
 			<geometry>
-				<mesh filename="file://$(find fiveages_body_description)/meshes/link3.glb"/>
+				<mesh filename="file://$(find fiveages_w2_description)/meshes/body/link3.glb"/>
 			</geometry>
 		</visual>
@@ -115,5 +115,5 @@
 		<child link="body_link3"/>
 		<axis xyz="0 1 0"/>
-		<limit lower="-1.745" upper="1.745" effort="500" velocity="1"/>
+		<limit lower="-${PI*50/180}" upper="${PI*70/180}" effort="100" velocity="1"/>
 	</joint>
 	<link name="body_link4">
@@ -131,5 +131,5 @@
 		<visual>
 			<geometry>
-				<mesh filename="file://$(find fiveages_body_description)/meshes/link4.glb"/>
+				<mesh filename="file://$(find fiveages_w2_description)/meshes/body/link4.glb"/>
 			</geometry>
 		</visual>
@@ -146,5 +146,5 @@
 		<child link="body_link4"/>
 		<axis xyz="0 0 -1"/>
-		<limit lower="-${PI}" upper="${PI}" effort="500" velocity="1"/>
+		<limit lower="-${PI}" upper="${PI}" effort="100" velocity="1"/>
 	</joint>
 	<link name="body_camera">
@@ -174,5 +174,5 @@
 		<visual>
 			<geometry>
-				<mesh filename="file://$(find fiveages_body_description)/meshes/head_yaw.glb"/>
+				<mesh filename="file://$(find fiveages_w2_description)/meshes/body/head_yaw.glb"/>
 			</geometry>
 		</visual>
@@ -183,5 +183,5 @@
 		<child link="head_link1"/>
 		<axis xyz="0 0 1"/>
-		<limit lower="-0.436" upper="0.436" effort="500" velocity="1"/>
+		<limit lower="-${PI*25/180}" upper="${PI*25/180}" effort="100" velocity="1"/>
 	</joint>
 	<link name="head_link2">
@@ -199,5 +199,5 @@
 		<visual>
 			<geometry>
-				<mesh filename="file://$(find fiveages_body_description)/meshes/head_pitch.glb"/>
+				<mesh filename="file://$(find fiveages_w2_description)/meshes/body/head_pitch.glb"/>
 			</geometry>
 		</visual>
@@ -214,5 +214,5 @@
 		<child link="head_link2"/>
 		<axis xyz="0 1 0"/>
-		<limit lower="-0.26" upper="0.26" effort="500" velocity="1"/>
+		<limit lower="-${PI*15/180}" upper="${PI*15/180}" effort="100" velocity="1"/>
 	</joint>
 	<link name="head_camera">
