Commit message: add variant

File: xacro/component.xacro (robot description, xacro)
@@ -4,7 +4,8 @@
 	<xacro:arg name="type" default="linkhou_s2_v2"/>
 	<xacro:arg name="chassis_joints_movable" default="true"/>
+	<xacro:arg name="variant" default=""/>
 	<xacro:if value="${'$(arg type)' == 'linkhou_s2'}">
 		<xacro:include filename="$(find fiveages_w2_common_description)/xacro/components/linkhou_s2.xacro"/>
-		<xacro:linkhou_s2 joints_movable="$(arg chassis_joints_movable)"/>
+		<xacro:linkhou_s2 joints_movable="$(arg chassis_joints_movable)" variant="$(arg variant)"/>
 	</xacro:if>
 	<xacro:if value="${'$(arg type)' == 'linkhou_s2_sinopec'}">
@@ -14,5 +15,5 @@
 	<xacro:if value="${'$(arg type)' == 'linkhou_s2_v2'}">
 		<xacro:include filename="$(find fiveages_w2_common_description)/xacro/components/linkhou_s2_v2.xacro"/>
-		<xacro:linkhou_s2 joints_movable="$(arg chassis_joints_movable)"/>
+		<xacro:linkhou_s2 joints_movable="$(arg chassis_joints_movable)" variant="$(arg variant)"/>
 	</xacro:if>
 	<xacro:if value="${'$(arg type)' == 'body'}">

File: xacro/components/linkhou_s2_v2.xacro (robot description, xacro)
@@ -2,5 +2,5 @@
 <robot name="FiveAges W2 Chassis" xmlns:xacro="http://www.ros.org/wiki/xacro">
 	<xacro:property name="PI" value="3.1415926535897931"/>
-	<xacro:macro name="linkhou_s2" params="joints_movable:=true">
+	<xacro:macro name="linkhou_s2" params="joints_movable:=true variant:=''">
 		<!-- 根据joints_movable参数设置关节类型 -->
 		<xacro:if value="${joints_movable}">
@@ -12,4 +12,6 @@
 			<xacro:property name="wheel_joint_type" value="fixed"/>
 		</xacro:unless>
+		<xacro:property name="shell_mesh" value="meshes/linkhou_s2_v2/shell_default.glb"/>
+		<xacro:property name="battery_mesh" value="meshes/linkhou_s2_v2/battery.glb"/>
 		<link name="base_footprint"/>
 		<joint name="base_footprint_joint" type="fixed">
@@ -43,5 +45,5 @@
 			<visual>
 				<geometry>
-					<mesh filename="file://$(find fiveages_w2_common_description)/meshes/linkhou_s2_v2/shell_default.glb"/>
+					<mesh filename="file://$(find fiveages_w2_common_description)/${shell_mesh}"/>
 				</geometry>
 			</visual>
@@ -378,5 +380,5 @@
 			<visual>
 				<geometry>
-					<mesh filename="file://$(find fiveages_w2_common_description)/meshes/linkhou_s2_v2/battery.glb"/>
+					<mesh filename="file://$(find fiveages_w2_common_description)/${battery_mesh}"/>
 				</geometry>
 			</visual>
@@ -390,5 +392,5 @@
 			<visual>
 				<geometry>
-					<mesh filename="file://$(find fiveages_w2_common_description)/meshes/linkhou_s2_v2/battery.glb"/>
+					<mesh filename="file://$(find fiveages_w2_common_description)/${battery_mesh}"/>
 				</geometry>
 			</visual>

Commit message: add body

File: xacro/component.xacro (robot description, xacro)
@@ -2,26 +2,42 @@
 <robot name="FiveAges W2" xmlns:xacro="http://www.ros.org/wiki/xacro">
 	<xacro:property name="PI" value="3.1415926535897931"/>
-	<!-- Component: linkhou_s2 (chassis), body, head. Chassis model via chassis:= ; OEM visuals via variant:= -->
+	<!-- Component: linkhou_s2 (chassis), body, head, stand, torso. Chassis model via chassis:= ; OEM visuals via variant:= -->
 	<xacro:arg name="type" default="linkhou_s2"/>
 	<xacro:arg name="chassis" default="linkhou_s2_v2"/>
 	<xacro:arg name="variant" default=""/>
+	<xacro:arg name="collider" default="simple"/>
 	<xacro:arg name="chassis_joints_movable" default="true"/>
 	<xacro:if value="${'$(arg type)' == 'linkhou_s2' and '$(arg chassis)' == 'linkhou_s2_v2'}">
 		<xacro:include filename="$(find fiveages_w2_common_description)/xacro/components/linkhou_s2_v2.xacro"/>
-		<xacro:linkhou_s2 joints_movable="$(arg chassis_joints_movable)" variant="$(arg variant)"/>
+		<xacro:linkhou_s2 joints_movable="$(arg chassis_joints_movable)" variant="$(arg variant)" collider="$(arg collider)"/>
 	</xacro:if>
 	<xacro:if value="${'$(arg type)' == 'linkhou_s2' and '$(arg chassis)' == 'linkhou_s2'}">
 		<xacro:include filename="$(find fiveages_w2_common_description)/xacro/components/linkhou_s2.xacro"/>
-		<xacro:linkhou_s2 joints_movable="$(arg chassis_joints_movable)" variant="$(arg variant)"/>
+		<xacro:linkhou_s2 joints_movable="$(arg chassis_joints_movable)" variant="$(arg variant)" collider="$(arg collider)"/>
 	</xacro:if>
 	<xacro:if value="${'$(arg type)' == 'body'}">
 		<link name="base_link"/>
 		<xacro:include filename="$(find fiveages_w2_common_description)/xacro/components/body.xacro"/>
-		<xacro:body variant="$(arg variant)"/>
+		<xacro:body variant="$(arg variant)" collider="$(arg collider)"/>
 	</xacro:if>
 	<xacro:if value="${'$(arg type)' == 'head'}">
 		<link name="head_mount"/>
 		<xacro:include filename="$(find fiveages_w2_common_description)/xacro/components/head.xacro"/>
-		<xacro:head variant="$(arg variant)"/>
+		<xacro:head variant="$(arg variant)" collider="$(arg collider)"/>
+	</xacro:if>
+	<xacro:if value="${'$(arg type)' == 'stand'}">
+		<xacro:include filename="$(find fiveages_w2_common_description)/xacro/components/stand.xacro"/>
+		<xacro:stand collider="$(arg collider)"/>
+	</xacro:if>
+	<xacro:if value="${'$(arg type)' == 'torso'}">
+		<link name="stand_link3"/>
+		<xacro:include filename="$(find fiveages_w2_common_description)/xacro/components/torso.xacro"/>
+		<xacro:torso
+				variant="$(arg variant)"
+				collider="$(arg collider)"
+				parent_link="stand_link3"
+				mount_joint_name="torso_mount_joint"
+				mount_joint_type="fixed"
+				mount_origin_xyz="-0.00076989 0 0.087931"/>
 	</xacro:if>
 </robot>

File: xacro/components/body.xacro (robot description, xacro)
@@ -2,5 +2,6 @@
 <robot name="FiveAges W2 Body" xmlns:xacro="http://www.ros.org/wiki/xacro">
 	<xacro:property name="PI" value="3.1415926535897931"/>
-	<xacro:macro name="body" params="variant:=''">
+	<xacro:include filename="$(find fiveages_w2_common_description)/xacro/components/torso.xacro"/>
+	<xacro:macro name="body" params="variant:='' collider:='simple'">
 		<xacro:property name="body_mesh_dir" value="meshes/body"/>
 		<xacro:property name="body_joint_effort" value="500"/>
@@ -40,4 +41,11 @@
 				</geometry>
 			</visual>
+			<xacro:if value="${collider == 'convex'}">
+				<collision>
+					<geometry>
+						<mesh filename="file://$(find fiveages_w2_common_description)/${body_mesh_dir}/base.glb"/>
+					</geometry>
+				</collision>
+			</xacro:if>
 		</link>
 		<joint name="body_fixed_joint" type="fixed">
@@ -63,10 +71,19 @@
 				</geometry>
 			</visual>
-			<collision>
-				<origin xyz="0.0 0 0.17"/>
-				<geometry>
-					<box size="0.15 0.145 0.48"/>
-				</geometry>
-			</collision>
+			<xacro:if value="${collider == 'simple'}">
+				<collision>
+					<origin xyz="0.0 0 0.17"/>
+					<geometry>
+						<box size="0.15 0.145 0.48"/>
+					</geometry>
+				</collision>
+			</xacro:if>
+			<xacro:if value="${collider == 'convex'}">
+				<collision>
+					<geometry>
+						<mesh filename="file://$(find fiveages_w2_common_description)/${body_mesh_dir}/link1.glb"/>
+					</geometry>
+				</collision>
+			</xacro:if>
 		</link>
 		<joint name="body_joint1" type="revolute">
@@ -93,10 +110,19 @@
 				</geometry>
 			</visual>
-			<collision>
-				<origin xyz="0.0 0 0.18"/>
-				<geometry>
-					<box size="0.16 0.2 0.5"/>
-				</geometry>
-			</collision>
+			<xacro:if value="${collider == 'simple'}">
+				<collision>
+					<origin xyz="0.0 0 0.18"/>
+					<geometry>
+						<box size="0.16 0.2 0.5"/>
+					</geometry>
+				</collision>
+			</xacro:if>
+			<xacro:if value="${collider == 'convex'}">
+				<collision>
+					<geometry>
+						<mesh filename="file://$(find fiveages_w2_common_description)/${body_mesh_dir}/link2.glb"/>
+					</geometry>
+				</collision>
+			</xacro:if>
 		</link>
 		<joint name="body_joint2" type="revolute">
@@ -124,10 +150,19 @@
 				</geometry>
 			</visual>
-			<collision>
-				<origin xyz="0.0 0 0.032"/>
-				<geometry>
-					<box size="0.13 0.13 0.22"/>
-				</geometry>
-			</collision>
+			<xacro:if value="${collider == 'simple'}">
+				<collision>
+					<origin xyz="0.0 0 0.032"/>
+					<geometry>
+						<box size="0.13 0.13 0.22"/>
+					</geometry>
+				</collision>
+			</xacro:if>
+			<xacro:if value="${collider == 'convex'}">
+				<collision>
+					<geometry>
+						<mesh filename="file://$(find fiveages_w2_common_description)/${body_mesh_dir}/link3.glb"/>
+					</geometry>
+				</collision>
+			</xacro:if>
 		</link>
 		<joint name="body_joint3" type="revolute">
@@ -138,59 +173,14 @@
 			<limit lower="${body_joint3_lower}" upper="${body_joint3_upper}" effort="${body_joint_effort}" velocity="1"/>
 		</joint>
-		<link name="body_link4">
-			<inertial>
-				<origin xyz="-0.0150844595179076 0.00261332042527829 0.274407850772391"/>
-				<mass value="23.7446394325596"/>
-				<inertia
-						ixx="0.320326293119484"
-						ixy="8.41740202015408E-05"
-						ixz="0.000603743723020676"
-						iyy="0.228575723449718"
-						iyz="8.78726038347342E-05"
-						izz="0.136416117968312"/>
-			</inertial>
-			<visual>
-				<geometry>
-					<mesh filename="file://$(find fiveages_w2_common_description)/${body_mesh_dir}/link4.glb"/>
-				</geometry>
-			</visual>
-			<collision>
-				<origin xyz="0.0091 0 0.25765"/>
-				<geometry>
-					<box size="0.2000 0.32 0.5029"/>
-				</geometry>
-			</collision>
-		</link>
-		<joint name="body_joint4" type="revolute">
-			<origin xyz="-7.1612E-05 -0.0019 0.14331"/>
-			<parent link="body_link3"/>
-			<child link="body_link4"/>
-			<axis xyz="0 0 -1"/>
-			<limit lower="${body_joint4_lower}" upper="${body_joint4_upper}" effort="${body_joint_effort}" velocity="1"/>
-		</joint>
-		<link name="body_camera">
-			<visual>
-				<geometry>
-					<mesh filename="file://$(find sensor_models)/meshes/orbbec/336.glb"/>
-				</geometry>
-			</visual>
-		</link>
-		<joint name="body_camera_joint" type="fixed">
-			<origin xyz="0.10065 0.024257 0.28812" rpy="${-PI/2-0.378684973} 0 ${-PI/2}"/>
-			<parent link="body_link4"/>
-			<child link="body_camera"/>
-		</joint>
-		<link name="head_mount"/>
-		<joint name="head_mount_joint" type="fixed">
-			<origin xyz="-0.023428 0 0.48475"/>
-			<parent link="body_link4"/>
-			<child link="head_mount"/>
-		</joint>
-		<link name="arm_base"/>
-		<joint name="arm_base_joint" type="fixed">
-			<origin xyz="7.1612E-05 0 0.45765"/>
-			<parent link="body_link4"/>
-			<child link="arm_base"/>
-		</joint>
+		<xacro:torso
+				variant="${variant}"
+				collider="${collider}"
+				parent_link="body_link3"
+				mount_joint_name="body_joint4"
+				mount_joint_type="revolute"
+				mount_origin_xyz="-7.1612E-05 -0.0019 0.14331"
+				mount_lower="${body_joint4_lower}"
+				mount_upper="${body_joint4_upper}"
+				mount_effort="${body_joint_effort}"/>
 	</xacro:macro>
 </robot>

File: xacro/components/head.xacro (robot description, xacro)
@@ -2,8 +2,20 @@
 <robot name="FiveAges W2 Head" xmlns:xacro="http://www.ros.org/wiki/xacro">
 	<xacro:property name="PI" value="3.1415926535897931"/>
-	<xacro:macro name="head" params="variant:=''">
+	<xacro:macro name="head" params="variant:='' collider:='simple'">
 		<xacro:property name="head_pitch_mesh" value="meshes/head/head_pitch.glb"/>
+		<!-- default: legacy W2 head limits -->
+		<xacro:property name="head_joint1_lower" value="-0.436"/>
+		<xacro:property name="head_joint1_upper" value="0.436"/>
+		<xacro:property name="head_joint2_lower" value="-0.26"/>
+		<xacro:property name="head_joint2_upper" value="0.26"/>
 		<xacro:if value="${variant == 'sinopec'}">
 			<xacro:property name="head_pitch_mesh" value="meshes/head/sinopec/head_pitch.glb"/>
+		</xacro:if>
+		<!-- stand / v1.5: LRAA0000000_0528_08.SLDASM.urdf joint05 & JOINT06 limits -->
+		<xacro:if value="${variant == 'stand' or variant == 'v1.5'}">
+			<xacro:property name="head_joint1_lower" value="-1.3963"/>
+			<xacro:property name="head_joint1_upper" value="1.3963"/>
+			<xacro:property name="head_joint2_lower" value="-0.4014"/>
+			<xacro:property name="head_joint2_upper" value="0.5236"/>
 		</xacro:if>
 		<link name="head_link1">
@@ -24,4 +36,11 @@
 				</geometry>
 			</visual>
+			<xacro:if value="${collider == 'convex'}">
+				<collision>
+					<geometry>
+						<mesh filename="file://$(find fiveages_w2_common_description)/meshes/head/head_yaw.glb"/>
+					</geometry>
+				</collision>
+			</xacro:if>
 		</link>
 		<!-- head_mount 与 head_link1 原点重合，偏航 DOF 在 head_joint1 -->
@@ -31,5 +50,5 @@
 			<child link="head_link1"/>
 			<axis xyz="0 0 1"/>
-			<limit lower="-0.436" upper="0.436" effort="500" velocity="1"/>
+			<limit lower="${head_joint1_lower}" upper="${head_joint1_upper}" effort="500" velocity="1"/>
 		</joint>
 		<link name="head_link2">
@@ -50,10 +69,24 @@
 				</geometry>
 			</visual>
-			<collision>
-				<origin xyz="0.025 0 0.04"/>
+			<visual>
 				<geometry>
-					<box size="0.15 0.16 0.24"/>
+					<mesh filename="file://$(find fiveages_w2_common_description)/meshes/head/neck.glb"/>
 				</geometry>
-			</collision>
+			</visual>
+			<xacro:if value="${collider == 'simple'}">
+				<collision>
+					<origin xyz="0.025 0 0.04"/>
+					<geometry>
+						<box size="0.15 0.16 0.24"/>
+					</geometry>
+				</collision>
+			</xacro:if>
+			<xacro:if value="${collider == 'convex'}">
+				<collision>
+					<geometry>
+						<mesh filename="file://$(find fiveages_w2_common_description)/${head_pitch_mesh}"/>
+					</geometry>
+				</collision>
+			</xacro:if>
 		</link>
 		<joint name="head_joint2" type="revolute">
@@ -62,5 +95,5 @@
 			<child link="head_link2"/>
 			<axis xyz="0 1 0"/>
-			<limit lower="-0.26" upper="0.26" effort="500" velocity="1"/>
+			<limit lower="${head_joint2_lower}" upper="${head_joint2_upper}" effort="500" velocity="1"/>
 		</joint>
 		<link name="head_camera">
@@ -72,5 +105,5 @@
 		</link>
 		<joint name="head_camera_joint" type="fixed">
-			<origin xyz="0.097847  0.046703 0.12364" rpy="${-PI/2-0.64460396} 0 ${-PI/2}"/>
+			<origin xyz="0.0976  0.043639 0.1243" rpy="${-PI/2-0.64460396} 0 ${-PI/2}"/>
 			<parent link="head_link2"/>
 			<child link="head_camera"/>

File: xacro/components/linkhou_s2.xacro (robot description, xacro)
@@ -2,5 +2,5 @@
 <robot name="FiveAges W2 Chassis" xmlns:xacro="http://www.ros.org/wiki/xacro">
 	<xacro:property name="PI" value="3.1415926535897931"/>
-	<xacro:macro name="linkhou_s2" params="joints_movable:=true variant:=''">
+	<xacro:macro name="linkhou_s2" params="joints_movable:=true variant:='' collider:='simple'">
 		<!-- 根据joints_movable参数设置关节类型 -->
 		<xacro:if value="${joints_movable}">
@@ -52,22 +52,36 @@
 				</geometry>
 			</visual>
-			<collision>
-				<origin xyz="0 0 0.15"/>
-				<geometry>
-					<box size="0.5 0.3 0.2"/>
-				</geometry>
-			</collision>
-			<collision>
-				<origin xyz="0 0.195 0.16"/>
-				<geometry>
-					<box size="0.66 0.16 0.3"/>
-				</geometry>
-			</collision>
-			<collision>
-				<origin xyz="0 -0.195 0.16"/>
-				<geometry>
-					<box size="0.66 0.16 0.3"/>
-				</geometry>
-			</collision>
+			<xacro:if value="${collider == 'simple'}">
+				<collision>
+					<origin xyz="0 0 0.15"/>
+					<geometry>
+						<box size="0.5 0.3 0.2"/>
+					</geometry>
+				</collision>
+				<collision>
+					<origin xyz="0 0.195 0.16"/>
+					<geometry>
+						<box size="0.66 0.16 0.3"/>
+					</geometry>
+				</collision>
+				<collision>
+					<origin xyz="0 -0.195 0.16"/>
+					<geometry>
+						<box size="0.66 0.16 0.3"/>
+					</geometry>
+				</collision>
+			</xacro:if>
+			<xacro:if value="${collider == 'convex'}">
+				<collision>
+					<geometry>
+						<mesh filename="file://$(find fiveages_w2_common_description)/meshes/linkhou_s2/base_link.glb"/>
+					</geometry>
+				</collision>
+				<collision>
+					<geometry>
+						<mesh filename="file://$(find fiveages_w2_common_description)/${shell_mesh}"/>
+					</geometry>
+				</collision>
+			</xacro:if>
 		</link>
 		<link name="rr_steer">

File: xacro/components/linkhou_s2_v2.xacro (robot description, xacro)
@@ -2,5 +2,5 @@
 <robot name="FiveAges W2 Chassis" xmlns:xacro="http://www.ros.org/wiki/xacro">
 	<xacro:property name="PI" value="3.1415926535897931"/>
-	<xacro:macro name="linkhou_s2" params="joints_movable:=true variant:=''">
+	<xacro:macro name="linkhou_s2" params="joints_movable:=true variant:='' collider:='simple'">
 		<!-- 根据joints_movable参数设置关节类型 -->
 		<xacro:if value="${joints_movable}">
@@ -48,22 +48,36 @@
 				</geometry>
 			</visual>
-			<collision>
-				<origin xyz="0 0 0.15"/>
-				<geometry>
-					<box size="0.5 0.3 0.2"/>
-				</geometry>
-			</collision>
-			<collision>
-				<origin xyz="0 0.195 0.16"/>
-				<geometry>
-					<box size="0.66 0.16 0.3"/>
-				</geometry>
-			</collision>
-			<collision>
-				<origin xyz="0 -0.195 0.16"/>
-				<geometry>
-					<box size="0.66 0.16 0.3"/>
-				</geometry>
-			</collision>
+			<xacro:if value="${collider == 'simple'}">
+				<collision>
+					<origin xyz="0 0 0.15"/>
+					<geometry>
+						<box size="0.5 0.3 0.2"/>
+					</geometry>
+				</collision>
+				<collision>
+					<origin xyz="0 0.195 0.16"/>
+					<geometry>
+						<box size="0.66 0.16 0.3"/>
+					</geometry>
+				</collision>
+				<collision>
+					<origin xyz="0 -0.195 0.16"/>
+					<geometry>
+						<box size="0.66 0.16 0.3"/>
+					</geometry>
+				</collision>
+			</xacro:if>
+			<xacro:if value="${collider == 'convex'}">
+				<collision>
+					<geometry>
+						<mesh filename="file://$(find fiveages_w2_common_description)/meshes/linkhou_s2_v2/base_link.glb"/>
+					</geometry>
+				</collision>
+				<collision>
+					<geometry>
+						<mesh filename="file://$(find fiveages_w2_common_description)/${shell_mesh}"/>
+					</geometry>
+				</collision>
+			</xacro:if>
 		</link>
 		<link name="rr_steer">

File: xacro/ros2_control/body.xacro (robot description, xacro)
@@ -40,3 +40,36 @@
     </joint>
   </xacro:macro>
+  <xacro:macro name="stand_interfaces">
+    <!-- body_joint1: prismatic lift [m]; body_joint2: revolute rotation [rad] -->
+    <joint name="body_joint1">
+      <command_interface name="position"/>
+      <state_interface name="position"/>
+      <state_interface name="velocity"/>
+      <state_interface name="effort"/>
+    </joint>
+    <joint name="body_joint2">
+      <command_interface name="position"/>
+      <state_interface name="position"/>
+      <state_interface name="velocity"/>
+      <state_interface name="effort"/>
+    </joint>
+    <joint name="body_joint3">
+      <command_interface name="position"/>
+      <state_interface name="position"/>
+      <state_interface name="velocity"/>
+      <state_interface name="effort"/>
+    </joint>
+    <joint name="head_joint1">
+      <command_interface name="position"/>
+      <state_interface name="position"/>
+      <state_interface name="velocity"/>
+      <state_interface name="effort"/>
+    </joint>
+    <joint name="head_joint2">
+      <command_interface name="position"/>
+      <state_interface name="position"/>
+      <state_interface name="velocity"/>
+      <state_interface name="effort"/>
+    </joint>
+  </xacro:macro>
 </robot>
