Commit message: add isaac support visualize param

File: xacro/component.xacro (robot description, xacro)
@@ -8,4 +8,5 @@
 	<xacro:arg name="collider" default="simple"/>
 	<xacro:arg name="chassis_joints_movable" default="true"/>
+	<xacro:arg name="isaac" default="false"/>
 	<xacro:if value="${'$(arg type)' == 'linkhou_s2' and '$(arg chassis)' == 'linkhou_s2_v2'}">
 		<xacro:include filename="$(find fiveages_w2_common_description)/xacro/components/linkhou_s2_v2.xacro"/>
@@ -19,10 +20,10 @@
 		<link name="base_link"/>
 		<xacro:include filename="$(find fiveages_w2_common_description)/xacro/components/body.xacro"/>
-		<xacro:body variant="$(arg variant)" collider="$(arg collider)"/>
+		<xacro:body variant="$(arg variant)" collider="$(arg collider)" isaac="$(arg isaac)"/>
 	</xacro:if>
 	<xacro:if value="${'$(arg type)' == 'head'}">
 		<link name="head_mount"/>
 		<xacro:include filename="$(find fiveages_w2_common_description)/xacro/components/head.xacro"/>
-		<xacro:head variant="$(arg variant)" collider="$(arg collider)"/>
+		<xacro:head variant="$(arg variant)" collider="$(arg collider)" isaac="$(arg isaac)"/>
 	</xacro:if>
 	<xacro:if value="${'$(arg type)' == 'stand'}">
@@ -36,4 +37,5 @@
 				variant="$(arg variant)"
 				collider="$(arg collider)"
+				isaac="$(arg isaac)"
 				parent_link="stand_link3"
 				mount_joint_name="torso_mount_joint"

File: xacro/components/body.xacro (robot description, xacro)
@@ -3,5 +3,5 @@
 	<xacro:property name="PI" value="3.1415926535897931"/>
 	<xacro:include filename="$(find fiveages_w2_common_description)/xacro/components/torso.xacro"/>
-	<xacro:macro name="body" params="variant:='' collider:='simple'">
+	<xacro:macro name="body" params="variant:='' collider:='simple' isaac:=false">
 		<xacro:property name="body_mesh_dir" value="meshes/body"/>
 		<xacro:property name="body_joint_effort" value="500"/>
@@ -176,4 +176,5 @@
 				variant="${variant}"
 				collider="${collider}"
+				isaac="${isaac}"
 				parent_link="body_link3"
 				mount_joint_name="body_joint4"

File: xacro/components/head.xacro (robot description, xacro)
@@ -2,5 +2,5 @@
 <robot name="FiveAges W2 Head" xmlns:xacro="http://www.ros.org/wiki/xacro">
 	<xacro:property name="PI" value="3.1415926535897931"/>
-	<xacro:macro name="head" params="variant:='' collider:='simple'">
+	<xacro:macro name="head" params="variant:='' collider:='simple' isaac:=false">
 		<xacro:property name="head_pitch_mesh" value="meshes/head/head_pitch.glb"/>
 		<!-- default: legacy W2 head limits -->
@@ -98,9 +98,11 @@
 		</joint>
 		<link name="head_camera">
-			<visual>
-				<geometry>
-					<mesh filename="file://$(find sensor_models)/meshes/orbbec/336L.glb"/>
-				</geometry>
-			</visual>
+			<xacro:unless value="${isaac}">
+				<visual>
+					<geometry>
+						<mesh filename="file://$(find sensor_models)/meshes/orbbec/336L.glb"/>
+					</geometry>
+				</visual>
+			</xacro:unless>
 		</link>
 		<joint name="head_camera_joint" type="fixed">

File: xacro/components/linkhou_s2.xacro (robot description, xacro)
@@ -2,5 +2,5 @@
 <robot name="FiveAges W2 Chassis" xmlns:xacro="http://www.ros.org/wiki/xacro">
 	<xacro:property name="PI" value="3.1415926535897931"/>
-	<xacro:macro name="linkhou_s2" params="joints_movable:=true variant:='' collider:='simple'">
+	<xacro:macro name="linkhou_s2" params="joints_movable:=true variant:='' collider:='simple' isaac:=false">
 		<!-- 根据joints_movable参数设置关节类型 -->
 		<xacro:if value="${joints_movable}">
@@ -47,9 +47,11 @@
 				</geometry>
 			</visual>
-			<visual>
-				<geometry>
-					<mesh filename="file://$(find fiveages_w2_common_description)/${shell_mesh}"/>
-				</geometry>
-			</visual>
+			<xacro:unless value="${isaac}">
+				<visual>
+					<geometry>
+						<mesh filename="file://$(find fiveages_w2_common_description)/${shell_mesh}"/>
+					</geometry>
+				</visual>
+			</xacro:unless>
 			<xacro:if value="${collider == 'simple'}">
 				<collision>
@@ -78,9 +80,11 @@
 					</geometry>
 				</collision>
-				<collision>
-					<geometry>
-						<mesh filename="file://$(find fiveages_w2_common_description)/${shell_mesh}"/>
-					</geometry>
-				</collision>
+				<xacro:unless value="${isaac}">
+					<collision>
+						<geometry>
+							<mesh filename="file://$(find fiveages_w2_common_description)/${shell_mesh}"/>
+						</geometry>
+					</collision>
+				</xacro:unless>
 			</xacro:if>
 		</link>
@@ -322,9 +326,11 @@
 		</joint>
 		<link name="rr_lidar">
-			<visual>
-				<geometry>
-					<mesh filename="file://$(find sensor_models)/meshes/robosense/airy.glb"/>
-				</geometry>
-			</visual>
+			<xacro:unless value="${isaac}">
+				<visual>
+					<geometry>
+						<mesh filename="file://$(find sensor_models)/meshes/robosense/airy.glb"/>
+					</geometry>
+				</visual>
+			</xacro:unless>
 		</link>
 		<joint name="rr_lidar_joint" type="fixed">
@@ -334,9 +340,11 @@
 		</joint>
 		<link name="fl_lidar">
-			<visual>
-				<geometry>
-					<mesh filename="file://$(find sensor_models)/meshes/robosense/airy.glb"/>
-				</geometry>
-			</visual>
+			<xacro:unless value="${isaac}">
+				<visual>
+					<geometry>
+						<mesh filename="file://$(find sensor_models)/meshes/robosense/airy.glb"/>
+					</geometry>
+				</visual>
+			</xacro:unless>
 		</link>
 		<joint name="fl_lidar_joint" type="fixed">
@@ -346,9 +354,11 @@
 		</joint>
 		<link name="chassis_camera">
-			<visual>
-				<geometry>
-					<mesh filename="file://$(find sensor_models)/meshes/linkhou/ds51.glb"/>
-				</geometry>
-			</visual>
+			<xacro:unless value="${isaac}">
+				<visual>
+					<geometry>
+						<mesh filename="file://$(find sensor_models)/meshes/linkhou/ds51.glb"/>
+					</geometry>
+				</visual>
+			</xacro:unless>
 		</link>
 		<joint name="chassis_camera_joint" type="fixed">
@@ -358,9 +368,11 @@
 		</joint>
 		<link name="chassis_left_battery">
-			<visual>
-				<geometry>
-					<mesh filename="file://$(find fiveages_w2_common_description)/${battery_mesh}"/>
-				</geometry>
-			</visual>
+			<xacro:unless value="${isaac}">
+				<visual>
+					<geometry>
+						<mesh filename="file://$(find fiveages_w2_common_description)/${battery_mesh}"/>
+					</geometry>
+				</visual>
+			</xacro:unless>
 		</link>
 		<joint name="chassis_left_battery" type="fixed">
@@ -370,9 +382,11 @@
 		</joint>
 		<link name="chassis_right_battery">
-			<visual>
-				<geometry>
-					<mesh filename="file://$(find fiveages_w2_common_description)/${battery_mesh}"/>
-				</geometry>
-			</visual>
+			<xacro:unless value="${isaac}">
+				<visual>
+					<geometry>
+						<mesh filename="file://$(find fiveages_w2_common_description)/${battery_mesh}"/>
+					</geometry>
+				</visual>
+			</xacro:unless>
 		</link>
 		<joint name="chassis_right_battery" type="fixed">
@@ -383,9 +397,11 @@
 		<!-- Ultrasonic sensors C1-C8 (poses from S2_3DURDF, mesh: sensor_models/ultrasonic_02) -->
 		<link name="ultrasonic_c1">
-			<visual>
-				<geometry>
-					<mesh filename="file://$(find sensor_models)/meshes/ultrasonic/ultrasonic_02.glb"/>
-				</geometry>
-			</visual>
+			<xacro:unless value="${isaac}">
+				<visual>
+					<geometry>
+						<mesh filename="file://$(find sensor_models)/meshes/ultrasonic/ultrasonic_02.glb"/>
+					</geometry>
+				</visual>
+			</xacro:unless>
 		</link>
 		<joint name="ultrasonic_c1_joint" type="fixed">
@@ -395,9 +411,11 @@
 		</joint>
 		<link name="ultrasonic_c2">
-			<visual>
-				<geometry>
-					<mesh filename="file://$(find sensor_models)/meshes/ultrasonic/ultrasonic_02.glb"/>
-				</geometry>
-			</visual>
+			<xacro:unless value="${isaac}">
+				<visual>
+					<geometry>
+						<mesh filename="file://$(find sensor_models)/meshes/ultrasonic/ultrasonic_02.glb"/>
+					</geometry>
+				</visual>
+			</xacro:unless>
 		</link>
 		<joint name="ultrasonic_c2_joint" type="fixed">
@@ -407,9 +425,11 @@
 		</joint>
 		<link name="ultrasonic_c3">
-			<visual>
-				<geometry>
-					<mesh filename="file://$(find sensor_models)/meshes/ultrasonic/ultrasonic_02.glb"/>
-				</geometry>
-			</visual>
+			<xacro:unless value="${isaac}">
+				<visual>
+					<geometry>
+						<mesh filename="file://$(find sensor_models)/meshes/ultrasonic/ultrasonic_02.glb"/>
+					</geometry>
+				</visual>
+			</xacro:unless>
 		</link>
 		<joint name="ultrasonic_c3_joint" type="fixed">
@@ -419,9 +439,11 @@
 		</joint>
 		<link name="ultrasonic_c4">
-			<visual>
-				<geometry>
-					<mesh filename="file://$(find sensor_models)/meshes/ultrasonic/ultrasonic_02.glb"/>
-				</geometry>
-			</visual>
+			<xacro:unless value="${isaac}">
+				<visual>
+					<geometry>
+						<mesh filename="file://$(find sensor_models)/meshes/ultrasonic/ultrasonic_02.glb"/>
+					</geometry>
+				</visual>
+			</xacro:unless>
 		</link>
 		<joint name="ultrasonic_c4_joint" type="fixed">
@@ -431,9 +453,11 @@
 		</joint>
 		<link name="ultrasonic_c5">
-			<visual>
-				<geometry>
-					<mesh filename="file://$(find sensor_models)/meshes/ultrasonic/ultrasonic_02.glb"/>
-				</geometry>
-			</visual>
+			<xacro:unless value="${isaac}">
+				<visual>
+					<geometry>
+						<mesh filename="file://$(find sensor_models)/meshes/ultrasonic/ultrasonic_02.glb"/>
+					</geometry>
+				</visual>
+			</xacro:unless>
 		</link>
 		<joint name="ultrasonic_c5_joint" type="fixed">
@@ -443,9 +467,11 @@
 		</joint>
 		<link name="ultrasonic_c6">
-			<visual>
-				<geometry>
-					<mesh filename="file://$(find sensor_models)/meshes/ultrasonic/ultrasonic_02.glb"/>
-				</geometry>
-			</visual>
+			<xacro:unless value="${isaac}">
+				<visual>
+					<geometry>
+						<mesh filename="file://$(find sensor_models)/meshes/ultrasonic/ultrasonic_02.glb"/>
+					</geometry>
+				</visual>
+			</xacro:unless>
 		</link>
 		<joint name="ultrasonic_c6_joint" type="fixed">
@@ -455,9 +481,11 @@
 		</joint>
 		<link name="ultrasonic_c7">
-			<visual>
-				<geometry>
-					<mesh filename="file://$(find sensor_models)/meshes/ultrasonic/ultrasonic_02.glb"/>
-				</geometry>
-			</visual>
+			<xacro:unless value="${isaac}">
+				<visual>
+					<geometry>
+						<mesh filename="file://$(find sensor_models)/meshes/ultrasonic/ultrasonic_02.glb"/>
+					</geometry>
+				</visual>
+			</xacro:unless>
 		</link>
 		<joint name="ultrasonic_c7_joint" type="fixed">
@@ -467,9 +495,11 @@
 		</joint>
 		<link name="ultrasonic_c8">
-			<visual>
-				<geometry>
-					<mesh filename="file://$(find sensor_models)/meshes/ultrasonic/ultrasonic_02.glb"/>
-				</geometry>
-			</visual>
+			<xacro:unless value="${isaac}">
+				<visual>
+					<geometry>
+						<mesh filename="file://$(find sensor_models)/meshes/ultrasonic/ultrasonic_02.glb"/>
+					</geometry>
+				</visual>
+			</xacro:unless>
 		</link>
 		<joint name="ultrasonic_c8_joint" type="fixed">

File: xacro/components/torso.xacro (robot description, xacro)
@@ -15,4 +15,5 @@
 		include_attachments:=true
 		collider:='simple'
+		isaac:=false
 	">
 		<link name="body_link4">
@@ -88,9 +89,11 @@
 		<xacro:if value="${include_attachments}">
 			<link name="body_camera1">
-				<visual>
-					<geometry>
-						<mesh filename="file://$(find sensor_models)/meshes/orbbec/336.glb"/>
-					</geometry>
-				</visual>
+				<xacro:unless value="${isaac}">
+					<visual>
+						<geometry>
+							<mesh filename="file://$(find sensor_models)/meshes/orbbec/336.glb"/>
+						</geometry>
+					</visual>
+				</xacro:unless>
 			</link>
 			<joint name="body_camera1_joint" type="fixed">
@@ -100,9 +103,11 @@
 			</joint>
 			<link name="body_camera2">
-				<visual>
-					<geometry>
-						<mesh filename="file://$(find sensor_models)/meshes/orbbec/336.glb"/>
-					</geometry>
-				</visual>
+				<xacro:unless value="${isaac}">
+					<visual>
+						<geometry>
+							<mesh filename="file://$(find sensor_models)/meshes/orbbec/336.glb"/>
+						</geometry>
+					</visual>
+				</xacro:unless>
 			</link>
 			<joint name="body_camera2_joint" type="fixed">

Commit message: update mesh

File: xacro/component.xacro (robot description, xacro)
@@ -29,5 +29,6 @@
 	<xacro:if value="${'$(arg type)' == 'stand'}">
 		<xacro:include filename="$(find fiveages_w2_common_description)/xacro/components/stand.xacro"/>
-		<xacro:stand collider="$(arg collider)"/>
+		<xacro:property name="lift_movable" value="${'$(arg variant)' != 'v0'}"/>
+		<xacro:stand collider="$(arg collider)" lift_movable="${lift_movable}"/>
 	</xacro:if>
 	<xacro:if value="${'$(arg type)' == 'torso'}">

File: xacro/components/stand.xacro (robot description, xacro)
@@ -3,5 +3,5 @@
 	<xacro:property name="PI" value="3.1415926535897931"/>
 	<xacro:property name="stand_mesh_dir" value="meshes/stand"/>
-	<xacro:macro name="stand" params="joint_effort:=100 collider:='simple'">
+	<xacro:macro name="stand" params="joint_effort:=100 collider:='simple' lift_movable:=true">
 		<link name="base_footprint"/>
 		<joint name="base_footprint_joint" type="fixed">
@@ -76,11 +76,20 @@
 			</xacro:if>
 		</link>
-		<joint name="body_joint1" type="prismatic">
-			<origin xyz="0 0 -0.188" rpy="0 0 0"/>
-			<parent link="base_link"/>
-			<child link="stand_link1"/>
-			<axis xyz="0 0 -1"/>
-			<limit lower="-0.1" upper="0.19" effort="${joint_effort}" velocity="1"/>
-		</joint>
+		<xacro:if value="${lift_movable}">
+			<joint name="lift_joint" type="prismatic">
+				<origin xyz="0 0 -0.188" rpy="0 0 0"/>
+				<parent link="base_link"/>
+				<child link="stand_link1"/>
+				<axis xyz="0 0 -1"/>
+				<limit lower="-0.1" upper="0.19" effort="${joint_effort}" velocity="1"/>
+			</joint>
+		</xacro:if>
+		<xacro:unless value="${lift_movable}">
+			<joint name="lift_joint" type="fixed">
+				<origin xyz="0 0 -0.188" rpy="0 0 0"/>
+				<parent link="base_link"/>
+				<child link="stand_link1"/>
+			</joint>
+		</xacro:unless>
 		<link name="stand_link2">
 			<inertial>
@@ -116,5 +125,5 @@
 			</xacro:if>
 		</link>
-		<joint name="body_joint2" type="revolute">
+		<joint name="body_joint1" type="revolute">
 			<origin xyz="0 0 0.547" rpy="0 0 0"/>
 			<parent link="stand_link1"/>
@@ -156,5 +165,5 @@
 			</xacro:if>
 		</link>
-		<joint name="body_joint3" type="revolute">
+		<joint name="body_joint2" type="revolute">
 			<origin xyz="0 0 0.116" rpy="0 0 0"/>
 			<parent link="stand_link2"/>

File: xacro/ros2_control/body.xacro (robot description, xacro)
@@ -40,6 +40,15 @@
     </joint>
   </xacro:macro>
-  <xacro:macro name="stand_interfaces">
-    <!-- body_joint1: prismatic lift [m]; body_joint2: revolute rotation [rad] -->
+  <xacro:macro name="stand_interfaces" params="lift_movable:=true">
+    <xacro:if value="${lift_movable}">
+      <!-- lift_joint: prismatic lift [m] -->
+      <joint name="lift_joint">
+        <command_interface name="position"/>
+        <state_interface name="position"/>
+        <state_interface name="velocity"/>
+        <state_interface name="effort"/>
+      </joint>
+    </xacro:if>
+    <!-- body_joint1: rotate [rad]; body_joint2: pitch [rad] -->
     <joint name="body_joint1">
       <command_interface name="position"/>
@@ -49,10 +58,4 @@
     </joint>
     <joint name="body_joint2">
-      <command_interface name="position"/>
-      <state_interface name="position"/>
-      <state_interface name="velocity"/>
-      <state_interface name="effort"/>
-    </joint>
-    <joint name="body_joint3">
       <command_interface name="position"/>
       <state_interface name="position"/>
