Commit message: fix linkhou s2 v2 shell mesh

File: xacro/component.xacro (robot description, xacro)
@@ -11,9 +11,9 @@
 	<xacro:if value="${'$(arg type)' == 'linkhou_s2' and '$(arg chassis)' == 'linkhou_s2_v2'}">
 		<xacro:include filename="$(find fiveages_w2_common_description)/xacro/components/linkhou_s2_v2.xacro"/>
-		<xacro:linkhou_s2 joints_movable="$(arg chassis_joints_movable)" variant="$(arg variant)" collider="$(arg collider)"/>
+		<xacro:linkhou_s2 joints_movable="$(arg chassis_joints_movable)" variant="$(arg variant)" collider="$(arg collider)" isaac="$(arg isaac)"/>
 	</xacro:if>
 	<xacro:if value="${'$(arg type)' == 'linkhou_s2' and '$(arg chassis)' == 'linkhou_s2'}">
 		<xacro:include filename="$(find fiveages_w2_common_description)/xacro/components/linkhou_s2.xacro"/>
-		<xacro:linkhou_s2 joints_movable="$(arg chassis_joints_movable)" variant="$(arg variant)" collider="$(arg collider)"/>
+		<xacro:linkhou_s2 joints_movable="$(arg chassis_joints_movable)" variant="$(arg variant)" collider="$(arg collider)" isaac="$(arg isaac)"/>
 	</xacro:if>
 	<xacro:if value="${'$(arg type)' == 'body'}">

File: xacro/components/linkhou_s2_v2.xacro (robot description, xacro)
@@ -2,5 +2,5 @@
 <robot name="FiveAges W2 Chassis" xmlns:xacro="http://www.ros.org/wiki/xacro">
 	<xacro:property name="PI" value="3.1415926535897931"/>
-	<xacro:macro name="linkhou_s2" params="joints_movable:=true variant:='' collider:='simple'">
+	<xacro:macro name="linkhou_s2" params="joints_movable:=true variant:='' collider:='simple' isaac:=false">
 		<!-- 根据joints_movable参数设置关节类型 -->
 		<xacro:if value="${joints_movable}">
@@ -43,9 +43,11 @@
 				</geometry>
 			</visual>
-			<visual>
-				<geometry>
-					<mesh filename="file://$(find fiveages_w2_common_description)/${shell_mesh}"/>
-				</geometry>
-			</visual>
+			<xacro:unless value="${isaac}">
+				<visual>
+					<geometry>
+						<mesh filename="file://$(find fiveages_w2_common_description)/${shell_mesh}"/>
+					</geometry>
+				</visual>
+			</xacro:unless>
 			<xacro:if value="${collider == 'simple'}">
 				<collision>
@@ -74,9 +76,11 @@
 					</geometry>
 				</collision>
-				<collision>
-					<geometry>
-						<mesh filename="file://$(find fiveages_w2_common_description)/${shell_mesh}"/>
-					</geometry>
-				</collision>
+				<xacro:unless value="${isaac}">
+					<collision>
+						<geometry>
+							<mesh filename="file://$(find fiveages_w2_common_description)/${shell_mesh}"/>
+						</geometry>
+					</collision>
+				</xacro:unless>
 			</xacro:if>
 		</link>
@@ -337,9 +341,11 @@
 						izz="5.88939528438811E-07"/>
 			</inertial>
-			<visual>
-				<geometry>
-					<mesh filename="file://$(find sensor_models)/meshes/livox/mid360.glb"/>
-				</geometry>
-			</visual>
+			<xacro:unless value="${isaac}">
+				<visual>
+					<geometry>
+						<mesh filename="file://$(find sensor_models)/meshes/livox/mid360.glb"/>
+					</geometry>
+				</visual>
+			</xacro:unless>
 		</link>
 		<joint name="rr_lidar_mount_joint" type="fixed">
@@ -368,9 +374,11 @@
 						izz="5.88939528438811E-07"/>
 			</inertial>
-			<visual>
-				<geometry>
-					<mesh filename="file://$(find sensor_models)/meshes/livox/mid360.glb"/>
-				</geometry>
-			</visual>
+			<xacro:unless value="${isaac}">
+				<visual>
+					<geometry>
+						<mesh filename="file://$(find sensor_models)/meshes/livox/mid360.glb"/>
+					</geometry>
+				</visual>
+			</xacro:unless>
 		</link>
 		<joint name="fl_lidar_mount_joint" type="fixed">
@@ -380,9 +388,11 @@
 		</joint>
 		<link name="chassis_camera">
-			<visual>
-				<geometry>
-					<mesh filename="file://$(find sensor_models)/meshes/linkhou/ds51.glb"/>
-				</geometry>
-			</visual>
+			<xacro:unless value="${isaac}">
+				<visual>
+					<geometry>
+						<mesh filename="file://$(find sensor_models)/meshes/linkhou/ds51.glb"/>
+					</geometry>
+				</visual>
+			</xacro:unless>
 		</link>
 		<joint name="chassis_camera_joint" type="fixed">
@@ -392,9 +402,11 @@
 		</joint>
 		<link name="chassis_left_battery">
-			<visual>
-				<geometry>
-					<mesh filename="file://$(find fiveages_w2_common_description)/${battery_mesh}"/>
-				</geometry>
-			</visual>
+			<xacro:unless value="${isaac}">
+				<visual>
+					<geometry>
+						<mesh filename="file://$(find fiveages_w2_common_description)/${battery_mesh}"/>
+					</geometry>
+				</visual>
+			</xacro:unless>
 		</link>
 		<joint name="chassis_left_battery" type="fixed">
@@ -404,9 +416,11 @@
 		</joint>
 		<link name="chassis_right_battery">
-			<visual>
-				<geometry>
-					<mesh filename="file://$(find fiveages_w2_common_description)/${battery_mesh}"/>
-				</geometry>
-			</visual>
+			<xacro:unless value="${isaac}">
+				<visual>
+					<geometry>
+						<mesh filename="file://$(find fiveages_w2_common_description)/${battery_mesh}"/>
+					</geometry>
+				</visual>
+			</xacro:unless>
 		</link>
 		<joint name="chassis_right_battery" type="fixed">
@@ -417,9 +431,11 @@
 		<!-- Ultrasonic sensors C1-C8 (poses from S2_3DURDF, mesh: sensor_models/ultrasonic_02) -->
 		<link name="ultrasonic_c1">
-			<visual>
-				<geometry>
-					<mesh filename="file://$(find sensor_models)/meshes/ultrasonic/ultrasonic_02.glb"/>
-				</geometry>
-			</visual>
+			<xacro:unless value="${isaac}">
+				<visual>
+					<geometry>
+						<mesh filename="file://$(find sensor_models)/meshes/ultrasonic/ultrasonic_02.glb"/>
+					</geometry>
+				</visual>
+			</xacro:unless>
 		</link>
 		<joint name="ultrasonic_c1_joint" type="fixed">
@@ -429,9 +445,11 @@
 		</joint>
 		<link name="ultrasonic_c2">
-			<visual>
-				<geometry>
-					<mesh filename="file://$(find sensor_models)/meshes/ultrasonic/ultrasonic_02.glb"/>
-				</geometry>
-			</visual>
+			<xacro:unless value="${isaac}">
+				<visual>
+					<geometry>
+						<mesh filename="file://$(find sensor_models)/meshes/ultrasonic/ultrasonic_02.glb"/>
+					</geometry>
+				</visual>
+			</xacro:unless>
 		</link>
 		<joint name="ultrasonic_c2_joint" type="fixed">
@@ -441,9 +459,11 @@
 		</joint>
 		<link name="ultrasonic_c3">
-			<visual>
-				<geometry>
-					<mesh filename="file://$(find sensor_models)/meshes/ultrasonic/ultrasonic_02.glb"/>
-				</geometry>
-			</visual>
+			<xacro:unless value="${isaac}">
+				<visual>
+					<geometry>
+						<mesh filename="file://$(find sensor_models)/meshes/ultrasonic/ultrasonic_02.glb"/>
+					</geometry>
+				</visual>
+			</xacro:unless>
 		</link>
 		<joint name="ultrasonic_c3_joint" type="fixed">
@@ -453,9 +473,11 @@
 		</joint>
 		<link name="ultrasonic_c4">
-			<visual>
-				<geometry>
-					<mesh filename="file://$(find sensor_models)/meshes/ultrasonic/ultrasonic_02.glb"/>
-				</geometry>
-			</visual>
+			<xacro:unless value="${isaac}">
+				<visual>
+					<geometry>
+						<mesh filename="file://$(find sensor_models)/meshes/ultrasonic/ultrasonic_02.glb"/>
+					</geometry>
+				</visual>
+			</xacro:unless>
 		</link>
 		<joint name="ultrasonic_c4_joint" type="fixed">
@@ -465,9 +487,11 @@
 		</joint>
 		<link name="ultrasonic_c5">
-			<visual>
-				<geometry>
-					<mesh filename="file://$(find sensor_models)/meshes/ultrasonic/ultrasonic_02.glb"/>
-				</geometry>
-			</visual>
+			<xacro:unless value="${isaac}">
+				<visual>
+					<geometry>
+						<mesh filename="file://$(find sensor_models)/meshes/ultrasonic/ultrasonic_02.glb"/>
+					</geometry>
+				</visual>
+			</xacro:unless>
 		</link>
 		<joint name="ultrasonic_c5_joint" type="fixed">
@@ -477,9 +501,11 @@
 		</joint>
 		<link name="ultrasonic_c6">
-			<visual>
-				<geometry>
-					<mesh filename="file://$(find sensor_models)/meshes/ultrasonic/ultrasonic_02.glb"/>
-				</geometry>
-			</visual>
+			<xacro:unless value="${isaac}">
+				<visual>
+					<geometry>
+						<mesh filename="file://$(find sensor_models)/meshes/ultrasonic/ultrasonic_02.glb"/>
+					</geometry>
+				</visual>
+			</xacro:unless>
 		</link>
 		<joint name="ultrasonic_c6_joint" type="fixed">
@@ -489,9 +515,11 @@
 		</joint>
 		<link name="ultrasonic_c7">
-			<visual>
-				<geometry>
-					<mesh filename="file://$(find sensor_models)/meshes/ultrasonic/ultrasonic_02.glb"/>
-				</geometry>
-			</visual>
+			<xacro:unless value="${isaac}">
+				<visual>
+					<geometry>
+						<mesh filename="file://$(find sensor_models)/meshes/ultrasonic/ultrasonic_02.glb"/>
+					</geometry>
+				</visual>
+			</xacro:unless>
 		</link>
 		<joint name="ultrasonic_c7_joint" type="fixed">
@@ -501,9 +529,11 @@
 		</joint>
 		<link name="ultrasonic_c8">
-			<visual>
-				<geometry>
-					<mesh filename="file://$(find sensor_models)/meshes/ultrasonic/ultrasonic_02.glb"/>
-				</geometry>
-			</visual>
+			<xacro:unless value="${isaac}">
+				<visual>
+					<geometry>
+						<mesh filename="file://$(find sensor_models)/meshes/ultrasonic/ultrasonic_02.glb"/>
+					</geometry>
+				</visual>
+			</xacro:unless>
 		</link>
 		<joint name="ultrasonic_c8_joint" type="fixed">

Commit message: add stand param

File: xacro/component.xacro (robot description, xacro)
@@ -8,5 +8,5 @@
 	<xacro:arg name="collider" default="simple"/>
 	<xacro:arg name="chassis_joints_movable" default="true"/>
-	<xacro:arg name="isaac" default="false"/>
+	<xacro:arg name="isaac" default="true"/>
 	<xacro:if value="${'$(arg type)' == 'linkhou_s2' and '$(arg chassis)' == 'linkhou_s2_v2'}">
 		<xacro:include filename="$(find fiveages_w2_common_description)/xacro/components/linkhou_s2_v2.xacro"/>

File: xacro/components/stand.xacro (robot description, xacro)
@@ -77,13 +77,15 @@
 		</link>
 		<xacro:if value="${lift_movable}">
+			<!-- q=0 fully down; q=0.29 fully up (axis +Z) -->
 			<joint name="lift_joint" type="prismatic">
-				<origin xyz="0 0 -0.188" rpy="0 0 0"/>
+				<origin xyz="0 0 -0.378" rpy="0 0 0"/>
 				<parent link="base_link"/>
 				<child link="stand_link1"/>
-				<axis xyz="0 0 -1"/>
-				<limit lower="-0.1" upper="0.19" effort="${joint_effort}" velocity="1"/>
+				<axis xyz="0 0 1"/>
+				<limit lower="0" upper="0.29" effort="${joint_effort}" velocity="1"/>
 			</joint>
 		</xacro:if>
 		<xacro:unless value="${lift_movable}">
+			<!-- Locked at former mid-travel height (equivalent to movable q=0.19) -->
 			<joint name="lift_joint" type="fixed">
 				<origin xyz="0 0 -0.188" rpy="0 0 0"/>

File: xacro/ros2_control/body.xacro (robot description, xacro)
@@ -42,5 +42,5 @@
   <xacro:macro name="stand_interfaces" params="lift_movable:=true">
     <xacro:if value="${lift_movable}">
-      <!-- lift_joint: prismatic lift [m] -->
+      <!-- lift_joint: prismatic lift [m]; 0=down, increase=up, range [0, 0.29] -->
       <joint name="lift_joint">
         <command_interface name="position"/>
