Commit message: add white skin

File: xacro/components/body.xacro (robot description, xacro)
@@ -23,4 +23,8 @@
 			<xacro:property name="body_joint3_lower" value="-${PI*50/180}"/>
 			<xacro:property name="body_joint3_upper" value="${PI*70/180}"/>
+		</xacro:if>
+		<xacro:property name="body_link2_mesh" value="${body_mesh_dir}/link2.glb"/>
+		<xacro:if value="${variant == 'white'}">
+			<xacro:property name="body_link2_mesh" value="meshes/body/white/link2.glb"/>
 		</xacro:if>
 		<link name="body_base">
@@ -107,5 +111,5 @@
 			<visual>
 				<geometry>
-					<mesh filename="file://$(find fiveages_w2_common_description)/${body_mesh_dir}/link2.glb"/>
+					<mesh filename="file://$(find fiveages_w2_common_description)/${body_link2_mesh}"/>
 				</geometry>
 			</visual>
@@ -121,5 +125,5 @@
 				<collision>
 					<geometry>
-						<mesh filename="file://$(find fiveages_w2_common_description)/${body_mesh_dir}/link2.glb"/>
+						<mesh filename="file://$(find fiveages_w2_common_description)/${body_link2_mesh}"/>
 					</geometry>
 				</collision>

File: xacro/components/head.xacro (robot description, xacro)
@@ -11,4 +11,7 @@
 		<xacro:if value="${variant == 'sinopec'}">
 			<xacro:property name="head_pitch_mesh" value="meshes/head/sinopec/head_pitch.glb"/>
+		</xacro:if>
+		<xacro:if value="${variant == 'white'}">
+			<xacro:property name="head_pitch_mesh" value="meshes/head/white/head_pitch.glb"/>
 		</xacro:if>
 		<!-- stand / v1.5: LRAA0000000_0528_08.SLDASM.urdf joint05 & JOINT06 limits -->

File: xacro/components/linkhou_s2_v2.xacro (robot description, xacro)
@@ -14,4 +14,8 @@
 		<xacro:property name="shell_mesh" value="meshes/linkhou_s2_v2/shell_default.glb"/>
 		<xacro:property name="battery_mesh" value="meshes/linkhou_s2_v2/battery.glb"/>
+		<xacro:if value="${variant == 'white'}">
+			<xacro:property name="shell_mesh" value="meshes/linkhou_s2_v2/white/shell.glb"/>
+			<xacro:property name="battery_mesh" value="meshes/linkhou_s2_v2/white/battery.glb"/>
+		</xacro:if>
 		<link name="base_footprint"/>
 		<joint name="base_footprint_joint" type="fixed">

File: xacro/components/torso.xacro (robot description, xacro)
@@ -29,10 +29,10 @@
 						izz="0.136416117968312"/>
 			</inertial>
+			<xacro:property name="torso_mesh" value="meshes/torso/torso.glb"/>
 			<xacro:if value="${variant == 'sinopec'}">
-				<visual>
-					<geometry>
-						<mesh filename="file://$(find fiveages_w2_common_description)/meshes/torso/sinopec/torso.glb"/>
-					</geometry>
-				</visual>
+				<xacro:property name="torso_mesh" value="meshes/torso/sinopec/torso.glb"/>
+			</xacro:if>
+			<xacro:if value="${variant == 'white'}">
+				<xacro:property name="torso_mesh" value="meshes/torso/white/torso.glb"/>
 			</xacro:if>
 			<xacro:unless value="${variant == 'sinopec'}">
@@ -42,10 +42,10 @@
 					</geometry>
 				</visual>
-				<visual>
-					<geometry>
-						<mesh filename="file://$(find fiveages_w2_common_description)/meshes/torso/torso.glb"/>
-					</geometry>
-				</visual>
 			</xacro:unless>
+			<visual>
+				<geometry>
+					<mesh filename="file://$(find fiveages_w2_common_description)/${torso_mesh}"/>
+				</geometry>
+			</visual>
 			<visual>
 				<geometry>
@@ -62,18 +62,9 @@
 			</xacro:if>
 			<xacro:if value="${collider == 'convex'}">
-				<xacro:if value="${variant == 'sinopec'}">
-					<collision>
-						<geometry>
-							<mesh filename="file://$(find fiveages_w2_common_description)/meshes/torso/sinopec/torso.glb"/>
-						</geometry>
-					</collision>
-				</xacro:if>
-				<xacro:unless value="${variant == 'sinopec'}">
-					<collision>
-						<geometry>
-							<mesh filename="file://$(find fiveages_w2_common_description)/meshes/torso/torso.glb"/>
-						</geometry>
-					</collision>
-				</xacro:unless>
+				<collision>
+					<geometry>
+						<mesh filename="file://$(find fiveages_w2_common_description)/${torso_mesh}"/>
+					</geometry>
+				</collision>
 			</xacro:if>
 		</link>
