Commit message: update collision geometry and positions in torso.xacro

File: xacro/components/torso.xacro (robot description, xacro)
@@ -55,7 +55,13 @@
 			<xacro:if value="${collider == 'simple'}">
 				<collision>
-					<origin xyz="0.0091 0 0.25765"/>
+					<origin xyz="0.0091 0 0.40"/>
 					<geometry>
-						<box size="0.2000 0.32 0.5029"/>
+						<box size="0.20 0.32 0.20"/>
+					</geometry>
+				</collision>
+				<collision>
+					<origin xyz="0.0091 0 0.15"/>
+					<geometry>
+						<box size="0.16 0.26 0.30"/>
 					</geometry>
 				</collision>

Commit message: refactor collision geometry in torso.xacro

File: xacro/components/torso.xacro (robot description, xacro)
@@ -54,10 +54,10 @@
 			</visual>
 			<xacro:if value="${collider == 'simple'}">
-				<collision>
+				<!-- <collision>
 					<origin xyz="0.0091 0 0.40"/>
 					<geometry>
-						<box size="0.20 0.32 0.20"/>
+						<box size="0.20 0.28 0.20"/>
 					</geometry>
-				</collision>
+				</collision> -->
 				<collision>
 					<origin xyz="0.0091 0 0.15"/>
