Commit message: 增加csv模式

File: xacro/ros2_control/body.xacro (robot description, xacro)
@@ -1,5 +1,9 @@
 <?xml version="1.0"?>
 <robot xmlns:xacro="http://www.ros.org/wiki/xacro">
-  <xacro:macro name="body_interfaces">
+  <xacro:macro name="body_interfaces" params="head_velocity:=false">
+    <xacro:waist_interfaces/>
+    <xacro:head_interfaces head_velocity="${head_velocity}"/>
+  </xacro:macro>
+  <xacro:macro name="waist_interfaces">
     <!-- 关节接口定义 -->
     <joint name="body_joint1">
@@ -27,6 +31,9 @@
        <state_interface name="effort"/>
     </joint>
+  </xacro:macro>
+  <xacro:macro name="head_interfaces" params="head_velocity:=true">
     <joint name="head_joint1">
       <command_interface name="position"/>
+      <xacro:if value="${head_velocity}"><command_interface name="velocity"/></xacro:if>
       <state_interface name="position"/>
       <state_interface name="velocity"/>
@@ -35,4 +42,5 @@
     <joint name="head_joint2">
       <command_interface name="position"/>
+      <xacro:if value="${head_velocity}"><command_interface name="velocity"/></xacro:if>
       <state_interface name="position"/>
       <state_interface name="velocity"/>

Commit message: 增加电流环速度参考接口

File: xacro/ros2_control/body.xacro (robot description, xacro)
@@ -1,12 +1,21 @@
 <?xml version="1.0"?>
 <robot xmlns:xacro="http://www.ros.org/wiki/xacro">
-  <xacro:macro name="body_interfaces" params="head_velocity:=false">
-    <xacro:waist_interfaces/>
-    <xacro:head_interfaces head_velocity="${head_velocity}"/>
+  <xacro:macro name="body_interfaces" params="waist_velocity:=false head_velocity:=false current_ids:=''">
+    <xacro:waist_interfaces waist_velocity="${waist_velocity}" current_ids="${current_ids}"/>
+    <xacro:head_interfaces head_velocity="${head_velocity}" current_ids="${current_ids}"/>
   </xacro:macro>
-  <xacro:macro name="waist_interfaces">
+  <!-- waist_velocity=true：4 个腰关节额外导出 velocity 命令口（Juxie CSV 模式必需，
+       否则 jx_hardware on_init 会抛 "CSV joint must declare a velocity command interface"）。
+       current_ids（如 "4"）：列出的电机也导出 velocity 命令口（**就是普通速度命令**）。
+       上层照旧只写 position(q_d)+velocity(q̇_d)；电流由驱动内部（0x05）按阻抗律算出 ——
+       区别只在驱动不把 velocity 转发给电机速度环，而是代进阻抗律当速度参考。
+       ⚠️ 电流环关节**不要**导出 effort：否则 CtrlInterfaces 的 MIX 自动检测会把整机切到 MIX。 -->
+  <xacro:macro name="waist_interfaces" params="waist_velocity:=false current_ids:=''">
+    <xacro:property name="body_current_ids"
+            value="${[v.strip() for v in str(current_ids).split(',') if v.strip()]}"/>
     <!-- 关节接口定义 -->
     <joint name="body_joint1">
       <command_interface name="position"/>
+      <xacro:if value="${waist_velocity or '1' in body_current_ids}"><command_interface name="velocity"/></xacro:if>
       <state_interface name="position"/>
       <state_interface name="velocity"/>
@@ -15,4 +24,5 @@
     <joint name="body_joint2">
       <command_interface name="position"/>
+      <xacro:if value="${waist_velocity or '2' in body_current_ids}"><command_interface name="velocity"/></xacro:if>
       <state_interface name="position"/>
       <state_interface name="velocity"/>
@@ -21,4 +31,5 @@
     <joint name="body_joint3">
       <command_interface name="position"/>
+      <xacro:if value="${waist_velocity or '3' in body_current_ids}"><command_interface name="velocity"/></xacro:if>
       <state_interface name="position"/>
       <state_interface name="velocity"/>
@@ -27,4 +38,5 @@
     <joint name="body_joint4">
       <command_interface name="position"/>
+      <xacro:if value="${waist_velocity or '4' in body_current_ids}"><command_interface name="velocity"/></xacro:if>
       <state_interface name="position"/>
       <state_interface name="velocity"/>
@@ -32,8 +44,10 @@
     </joint>
   </xacro:macro>
-  <xacro:macro name="head_interfaces" params="head_velocity:=true">
+  <xacro:macro name="head_interfaces" params="head_velocity:=true current_ids:=''">
+    <xacro:property name="head_current_ids"
+            value="${[v.strip() for v in str(current_ids).split(',') if v.strip()]}"/>
     <joint name="head_joint1">
       <command_interface name="position"/>
-      <xacro:if value="${head_velocity}"><command_interface name="velocity"/></xacro:if>
+      <xacro:if value="${head_velocity or '5' in head_current_ids}"><command_interface name="velocity"/></xacro:if>
       <state_interface name="position"/>
       <state_interface name="velocity"/>
@@ -42,5 +56,5 @@
     <joint name="head_joint2">
       <command_interface name="position"/>
-      <xacro:if value="${head_velocity}"><command_interface name="velocity"/></xacro:if>
+      <xacro:if value="${head_velocity or '6' in head_current_ids}"><command_interface name="velocity"/></xacro:if>
       <state_interface name="position"/>
       <state_interface name="velocity"/>
